File: sbc-av/sbc-av.kicad_pcb (KiCad board)
At the start: 4 copper layers, 17.8 x 38.1 mm, 42 parts, among them J1 AVD-Header, J2 AVA-Header, Q1 PZT2222A, U1 MAX1683, U2 CD74HCT367E, U3 FMS6400

Commit message: WIP: sbc-sv 1.2
Parts:
- removed D1: BAT48JFILM, Diode_SMD:D_SOD-323_HandSoldering
- added C14: 47pF, Capacitor_SMD:C_0805_2012Metric_Pad1.18x1.45mm_HandSolder, F.Cu at (135.3, 66.0)
- added C15: 10uF, Capacitor_Tantalum_SMD:CP_EIA-3216-18_Kemet-A_HandSolder, F.Cu at (135.3, 61.0)
- added Q2: 2N7002, Package_TO_SOT_SMD:SOT-23, F.Cu at (130.4, 75.6)
- added R12: 4K20, Resistor_SMD:R_0805_2012Metric_Pad1.20x1.40mm_HandSolder, F.Cu at (125.7, 75.6)
- added R23: 10K, Resistor_SMD:R_0805_2012Metric_Pad1.20x1.40mm_HandSolder, F.Cu at (135.3, 69.8)
- added R24: 100R, Resistor_SMD:R_0805_2012Metric_Pad1.20x1.40mm_HandSolder, F.Cu at (137.8, 60.3)
- added U4: OPA134, Package_SO:SOIC-8_3.9x4.9mm_P1.27mm, F.Cu at (139.1, 66.0)
- C11: value 0.1uF -> 10uF; footprint Capacitor_SMD:C_0805_2012Metric_Pad1.18x1.45mm_HandSolder -> Capacitor_Tantalum_SMD:CP_EIA-2012-15_AVX-P_HandSolder
- C12: value 0.1uF -> 0.22uF; footprint Capacitor_SMD:C_0805_2012Metric_Pad1.18x1.45mm_HandSolder -> Capacitor_SMD:C_1206_3216Metric_Pad1.33x1.80mm_HandSolder; moved to B.Cu
- C13: value 10uF -> 0.22uF; footprint Capacitor_SMD:C_0805_2012Metric_Pad1.18x1.45mm_HandSolder -> Capacitor_SMD:C_1206_3216Metric_Pad1.33x1.80mm_HandSolder; moved to B.Cu
- C4: value 10uF -> 0.1uF
- C5: value 3.3uF -> 10uF; footprint Capacitor_SMD:C_0805_2012Metric_Pad1.18x1.45mm_HandSolder -> Capacitor_Tantalum_SMD:CP_EIA-2012-15_AVX-P_HandSolder; moved to F.Cu
- C7: value 0.1uF -> 3.3uF
- C8: moved to B.Cu
- C9: value 100pF -> 0.1uF
- Q1: value PZT2222A -> 2N7002; footprint Package_TO_SOT_SMD:SOT-223-3_TabPin2 -> Package_TO_SOT_SMD:SOT-23
- R10, R16, R9: value 75R -> 1K
- R11: value 75R -> 499R
- R13: value 1K -> 287R
- R14: value 180R -> 3K
- R15: value 150R -> 4K99
- R17: value 100K -> 75R
- R18: value 470K -> 75R
- R20: value 75R -> 10K
- R21: value 75R -> 47K; moved to B.Cu
- R22: value 75R -> 220K; moved to B.Cu
- R3, R4, R5, R6, R7: value 150R -> 2K
- R8: value 150R -> 1K
- U3: value FMS6400 -> THS7316
- moved C5 23.4 mm to (131.4, 61.0), turned to -90 degrees
- moved R17 18.0 mm to (126.4, 60.3)
- moved C12 16.7 mm to (141.0, 61.0), turned to -90 degrees
- moved R21 15.9 mm to (141.0, 65.4), turned to -90 degrees
- moved R18 15.1 mm to (128.9, 60.3)
- moved Q1 12.8 mm to (134.3, 79.4), turned to 90 degrees
- moved R19 11.4 mm to (137.2, 71.8), turned to -90 degrees
- moved R20 11.3 mm to (139.1, 71.8), turned to 90 degrees
- moved R2 10.7 mm to (140.8, 84.3), turned to -90 degrees
- moved C8 10.6 mm to (135.9, 75.6), turned to -90 degrees
- moved C9 9.44 mm to (125.7, 71.8), turned to 90 degrees
- moved R22 8.82 mm to (138.4, 65.4), turned to -90 degrees
- moved C1 7.64 mm to (139.8, 76.2), turned to 0 degrees
- moved R1 7.36 mm to (138.6, 84.3), turned to 90 degrees
- moved C4 7.01 mm to (140.3, 60.3)
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Connections:
- C10 pad 2: Net-(U3-CIN) -> Net-(U3-CH3.IN)
- C11 pad 1: POKEY_AUDIO -> Net-(U4-+)
- C11 pad 2: Net-(C11-Pad2) -> GND
- C12 pad 1: GTIA_AUDIO -> POKEY_AUDIO
- C13 pad 1: Net-(Q1-C) -> GTIA_AUDIO
- C13 pad 2: AUDIO_OUT -> Net-(C13-Pad2)
- C5 pad 1: Net-(U1-C1+) -> +5V
- C5 pad 2: Net-(U1-C1-) -> GND
- C6 pad 1: Net-(U1-OUT) -> Net-(U1-C1+)
- C6 pad 2: GND -> Net-(U1-C1-)
- C7 pad 1: CADJ -> Net-(U1-OUT)
- C8 pad 1: Net-(C8-Pad1) -> CADJ
- C8 pad 2: Net-(U3-YIN) -> GND
- C9 pad 1: COLOR -> Net-(Q2-D)
- C9 pad 2: Net-(C9-Pad2) -> Net-(U3-CH1.IN)
- Q1 pad 1: Net-(Q1-B) -> CSYNCB
- Q1 pad 2: Net-(Q1-C) -> GND
- Q1 pad 3: GND -> Net-(Q1-D)
- R11 pad 2: Net-(D1-A) -> Net-(Q2-D)
- R13 pad 1: Net-(D1-A) -> GND
- R13 pad 2: Net-(C8-Pad1) -> Net-(Q2-D)
- R14 pad 1: Net-(C8-Pad1) -> Net-(Q1-D)
- R14 pad 2: GND -> +5V
- R15 pad 1: GND -> COLOR
- R15 pad 2: Net-(C9-Pad2) -> Net-(C10-Pad1)
- R16 pad 1: Net-(C9-Pad2) -> GND
- R17 pad 1: Net-(C11-Pad2) -> Net-(U3-CH1.OUT)
- R17 pad 2: Net-(Q1-B) -> SVIDEO_Y
- R18 pad 1: Net-(C12-Pad2) -> Net-(U3-CH3.OUT)
- R18 pad 2: Net-(Q1-B) -> SVIDEO_C
- R19 pad 1: Net-(Q1-B) -> Net-(U4-+)
- R19 pad 2: Net-(Q1-C) -> +5V
- R20 pad 1: +5V -> GND
- R20 pad 2: Net-(Q1-C) -> Net-(U4-+)
- R21 pad 1: Net-(U3-YOUT) -> Net-(C12-Pad2)
- R21 pad 2: SVIDEO_Y -> Net-(U4--)
- R22 pad 1: Net-(U3-COUT) -> Net-(C13-Pad2)
- R22 pad 2: SVIDEO_C -> Net-(U4--)
- R3 pad 1: Net-(R3-Pad1) -> GND
- R3 pad 2: GND -> Net-(R3-Pad2)
- R4 pad 1: Net-(R3-Pad1) -> Net-(R3-Pad2)
- R5 pad 1: Net-(R10-Pad1) -> Net-(R5-Pad1)
- R6 pad 1: Net-(R10-Pad2) -> Net-(R10-Pad1)
- R7 pad 1: Net-(D1-A) -> Net-(R10-Pad2)
- R8 pad 1: Net-(D1-A) -> Net-(R3-Pad2)
- R8 pad 2: +5V -> Net-(R5-Pad1)
- R9 pad 1: Net-(R3-Pad1) -> Net-(R5-Pad1)
- U3 pad 1: Net-(U3-YIN) -> Net-(U3-CH1.IN)
- U3 pad 3: GND -> Net-(U3-CH3.IN)
- U3 pad 4: Net-(U3-CIN) -> +5V
- U3 pad 5: Net-(U3-COUT) -> GND
- U3 pad 6: unconnected-(U3-CVOUT-Pad6) -> Net-(U3-CH3.OUT)
- U3 pad 7: +5V -> unconnected-(U3-CH2.OUT-Pad7)
- U3 pad 8: Net-(U3-YOUT) -> Net-(U3-CH1.OUT)
Routing:
- net GTIA_AUDIO: track 44.2 -> 14.8 mm
- net POKEY_AUDIO: track 24.0 -> 5.31 mm, vias 1 -> 0
- net Net-(Q1-B): track 14.6 -> 0.00 mm
- net Net-(Q1-C): track 13.8 -> 0.00 mm
- net Net-(U4--): track 0.00 -> 13.4 mm, vias 0 -> 1
- net Net-(D1-A): track 12.9 -> 0.00 mm
- net Net-(C14-Pad2): track 0.00 -> 12.8 mm
- net Net-(Q2-D): track 0.00 -> 9.67 mm
- net Net-(U1-C1-): track 10.9 -> 2.07 mm
- net COLOR: track 12.5 -> 19.7 mm, vias 1 -> 2
- net Net-(C9-Pad2): track 6.85 -> 0.00 mm
- net Net-(U4-+): track 0.00 -> 6.32 mm
- net Net-(R3-Pad1): track 6.12 -> 0.00 mm
- net CADJ: track 30.9 -> 24.9 mm
- net Net-(R5-Pad1): track 0.00 -> 6.02 mm
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Other:
- board text added: "SFF AV v1.2 © 2026 Daniel Picken github.com/dpicken/atari-hw"
- board text removed: "SFF AV v1.1 © 2023 Daniel Picken github.com/dpicken/atari-hw"
