File: sbc-av/sbc-av.kicad_sch (KiCad schematic)
At the start: 42 parts, among them J1 AVD-Header, J2 AVA-Header, Q1 PZT2222A, U1 MAX1683, U2 CD74HCT367E, U3 FMS6400

Commit message: WIP: sbc-sv 1.2
Parts:
- removed C11: 0.1uF, Capacitor_SMD:C_0805_2012Metric_Pad1.18x1.45mm_HandSolder, symbol Device:C
- removed C9: 100pF, Capacitor_SMD:C_0805_2012Metric_Pad1.18x1.45mm_HandSolder, symbol Device:C
- removed D1: BAT48JFILM, Diode_SMD:D_SOD-323_HandSoldering, symbol Diode:BAT48JFILM
- removed Q1: PZT2222A, Package_TO_SOT_SMD:SOT-223-3_TabPin2, symbol Transistor_BJT:PZT2222A
- removed R17: 100K, Resistor_SMD:R_0805_2012Metric_Pad1.20x1.40mm_HandSolder, symbol Device:R
- removed R18: 470K, Resistor_SMD:R_0805_2012Metric_Pad1.20x1.40mm_HandSolder, symbol Device:R
- removed U3: FMS6400, Package_SO:SOIC-8_3.9x4.9mm_P1.27mm, symbol Project_Amplifier_Video:FMS6400
- added C11, C5: 10uF, Capacitor_Tantalum_SMD:CP_EIA-2012-15_AVX-P_HandSolder, symbol Device:C_Polarized_US
- added C14: 47pF, Capacitor_SMD:C_0805_2012Metric_Pad1.18x1.45mm_HandSolder, symbol Device:C
- added C15: 10uF, Capacitor_Tantalum_SMD:CP_EIA-3216-18_Kemet-A_HandSolder, symbol Device:C_Polarized_US
- added Q1, Q2: 2N7002, Package_TO_SOT_SMD:SOT-23, symbol Transistor_FET:2N7002
- added R11: 499R, Resistor_SMD:R_0805_2012Metric_Pad1.20x1.40mm_HandSolder, symbol Device:R
- added R21: 47K, Resistor_SMD:R_0805_2012Metric_Pad1.20x1.40mm_HandSolder, symbol Device:R
- added R22: 220K, Resistor_SMD:R_0805_2012Metric_Pad1.20x1.40mm_HandSolder, symbol Device:R
- added R23: 10K, Resistor_SMD:R_0805_2012Metric_Pad1.20x1.40mm_HandSolder, symbol Device:R
- added R24: 100R, Resistor_SMD:R_0805_2012Metric_Pad1.20x1.40mm_HandSolder, symbol Device:R
- added U3: THS7316, Package_SO:SOIC-8_3.9x4.9mm_P1.27mm, symbol Project_Amplifier_Video:THS7316
- added U4: OPA134, Package_SO:SOIC-8_3.9x4.9mm_P1.27mm, symbol Amplifier_Operational:OPA134
- C12: value 0.1uF -> 0.22uF; footprint Capacitor_SMD:C_0805_2012Metric_Pad1.18x1.45mm_HandSolder -> Capacitor_SMD:C_1206_3216Metric_Pad1.33x1.80mm_HandSolder
- C13: value 10uF -> 0.22uF; footprint Capacitor_SMD:C_0805_2012Metric_Pad1.18x1.45mm_HandSolder -> Capacitor_SMD:C_1206_3216Metric_Pad1.33x1.80mm_HandSolder
- C4: value 10uF -> 0.1uF
- R10: renamed from R11; value 75R -> 1K
- R12: renamed from R8; value 150R -> 4K20
- R13: value 1K -> 287R
- R14: value 180R -> 3K
- R15: renamed from R16; value 75R -> 4K99
- R16: renamed from R15; value 150R -> 1K
- R20: value 75R -> 10K
- R3, R4, R5, R6, R7: value 150R -> 2K
- R8: renamed from R9; value 75R -> 1K
- R9: renamed from R10; value 75R -> 1K
- renumbered C5 to C6, C6 to C7, C7 to C8, C8 to C9, R21 to R17, R22 to R18
Connections:
- net +5V: now also R14.2, R19.2, C5.1, U3.4 (VS+), U4.7 (V+); no longer R20.1
- net AUDIO_OUT: now also R24.2; no longer C13.2
- net COLOR: now also R15.1
- net CSYNCB: now also Q1.1 (G)
- net GND: now also R13.1, R20.1, R3.1, C11.2, C5.2, Q1.2 (S), Q2.2 (S), U3.2 (CH2.IN), U3.5 (GND), U4.4 (V-); no longer R14.2, R3.2
- net GTIA_AUDIO: now also C13.1; no longer C12.1
- net POKEY_AUDIO: now also C12.1
- net at R16.2: now also C10.1, R15.2; no longer R15.1
- net at R10.2, R7.1: now also R11.1; no longer R12.1, R13.1
- net at C9.1, R13.2: now also R12.1, Q2.3 (D), R11.2; no longer R14.1
- net at C10.2: now also U3.3 (CH3.IN)
- net at R4.1, R8.1: now also R3.2; no longer R3.1
- net at R19.1: now also R20.2, C11.1, U4.3 (+)
- net at C9.2: now also U3.1 (CH1.IN)
- net at C12.2: now also R21.1
- net at R18.1: now also U3.6 (CH3.OUT)
- net at R17.1: now also U3.8 (CH1.OUT)
- new net: C14.1, R21.2, R22.2, R23.1, U4.2 (-)
- new net: C14.2, C15.1, R23.2, U4.6
- new net: Q1.3 (D), Q2.1 (G), R14.1
- new net: C13.2, R22.1
- new net: C15.2, R24.1
- no-connect marks 3 -> 5
Other:
- moved on the sheet: C1, C10, C2, C3, C9, R10, R12, R15, R16, R17, R18, R3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
